File: Hardware/power_v1.0/power_v1.0.kicad_sch (KiCad schematic)
At the start: 5 parts, among them J4 Conn_01x02

Commit message: finished part selection for power and almost done with part selection for brain--moving to layout next
Parts:
- added C22, C26, C27, C29, C33, C34, C36, C40, C41: 22uF, Capacitor_SMD:C_0805_2012Metric, symbol Device:C_Small
- added C23, C25, C30, C32, C37, C39: 0.1uF, Capacitor_SMD:C_0603_1608Metric, symbol Device:C_Small
- added C24, C31, C38: 22nF, Capacitor_SMD:C_0805_2012Metric, symbol Device:C_Small
- added C28, C35, C42: 300pF, Capacitor_SMD:C_0805_2012Metric, symbol Device:C_Small
- added D1, D2, D3, D4, D5, D6: D_Schottky, VS_30BQ015_M3_9AT:VS_30BQ015_M3_9AT, symbol Device:D_Schottky
- added F1, F2, F3: Fuse, 4628:FUSE_4628, symbol Device:Fuse
- added J5: Motor1_Power, Connector_Molex:Molex_KK-254_AE-6410-02A_1x02_P2.54mm_Vertical, symbol Connector_Generic:Conn_01x02
- added J6: Sensor_Power, Connector_Molex:Molex_KK-254_AE-6410-02A_1x02_P2.54mm_Vertical, symbol Connector_Generic:Conn_01x02
- added J7: Motor2_Power, Connector_Molex:Molex_KK-254_AE-6410-02A_1x02_P2.54mm_Vertical, symbol Connector_Generic:Conn_01x02
- added JP1, JP2, JP3: SolderJumper_2_Bridged, Jumper:SolderJumper-2_P1.3mm_Bridged_RoundedPad1.0x1.5mm, symbol Jumper:SolderJumper_2_Bridged
- added L1, L2, L3: 6.8uH, 7447786006:WE-PD_6050R, symbol device:L
- added R22, R29, R36: 191k, Resistor_SMD:R_1210_3225Metric, symbol Device:R_US
- added R23, R30, R37: 49.9k, Resistor_SMD:R_2512_6332Metric, symbol Device:R_US
- added R24, R25, R27, R31, R32, R34, R38, R39, R41: 10k, Resistor_SMD:R_1206_3216Metric, symbol Device:R_US
- added R26, R33, R40: 90.9k, Resistor_SMD:R_1206_3216Metric, symbol Device:R_US
- added R28, R35, R42: 100k, Resistor_SMD:R_0805_2012Metric, symbol Device:R_US
- added TP1: 12V, TestPoint:TestPoint_Keystone_5010-5014_Multipurpose, symbol Connector:TestPoint
- added TP2: GND, TestPoint:TestPoint_Keystone_5010-5014_Multipurpose, symbol Connector:TestPoint
- added TP3: Motor2_Power, TestPoint:TestPoint_Keystone_5010-5014_Multipurpose, symbol Connector:TestPoint
- added TP4: Motor1_Power, TestPoint:TestPoint_Keystone_5010-5014_Multipurpose, symbol Connector:TestPoint
- added TP5: Sensor_Power, TestPoint:TestPoint_Keystone_5010-5014_Multipurpose, symbol Connector:TestPoint
- added U4, U5, U6: MP2338GTL-Z, SOT583_MP2338_MNP, symbol MP2338GTL-Z:MP2338GTL-Z
- H1, H2, H3, H4: footprint (none) -> MountingHole:MountingHole_3.2mm_M3; Link (none) -> NA; MPN (none) -> NA
- J4: value Conn_01x02 -> 12V IN; footprint (none) -> Connector_Molex:Molex_KK-254_AE-6410-02A_1x02_P2.54mm_Vertical; Link (none) -> https://www.digikey.com/en/products/detail/molex/1718560102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; MPN (none) -> 1718560102
Connections:
- net +12V: now also F1.1, F2.1, F3.1, TP1.1
- net GND: now also C22.2, C23.2, C26.2, C27.2, C29.2, C30.2, C33.2, C34.2, C36.2, C37.2, C40.2, C41.2, J5.2 (Pin_2), J6.2 (Pin_2), J7.2 (Pin_2), R23.2, R27.2, R28.2, R30.2, R34.2, R35.2, R37.2, R41.2, R42.2, TP2.1
- new net: C38.1, U6.4 (GND)
- new net: C38.2, U6.7 (SS)
- new net: C26.1, C27.1, C28.1, JP2.1 (A), L2.2, R24.2, R26.1, R28.1, TP4.1
- new net: C28.2, R25.2, R26.2, R27.1
- new net: R31.1, U5.1 (PG)
- new net: C29.1, C30.1, D1.1 (K), R29.1, U5.2 (VIN)
- new net: C32.2, U5.3 (SW)
- new net: C31.1, U5.4 (GND)
- new net: C32.1, L1.1, U5.5 (BST)
- new net: R29.2, R30.1, U5.6 (EN)
- new net: C31.2, U5.7 (SS)
- new net: R32.1, U5.8 (FB)
- new net: C22.1, C23.1, D2.1 (K), R22.1, U4.2 (VIN)
- new net: D2.2 (A), F2.2
- new net: D5.2 (A), JP2.2 (B)
- new net: C33.1, C34.1, C35.1, JP1.1 (A), L1.2, R31.2, R33.1, R35.1, TP5.1
- new net: C25.1, L2.1, U4.5 (BST)
- new net: C40.1, C41.1, C42.1, JP3.1 (A), L3.2, R38.2, R40.1, R42.1, TP3.1
- new net: C42.2, R39.2, R40.2, R41.1
- new net: D6.1 (K), J7.1 (Pin_1)
- new net: D6.2 (A), JP3.2 (B)
- new net: C25.2, U4.3 (SW)
- new net: D5.1 (K), J5.1 (Pin_1)
- new net: R22.2, R23.1, U4.6 (EN)
- new net: R24.1, U4.1 (PG)
- new net: C35.2, R32.2, R33.2, R34.1
- new net: D4.1 (K), J6.1 (Pin_1)
- new net: C39.1, L3.1, U6.5 (BST)
- new net: C39.2, U6.3 (SW)
- new net: R36.2, R37.1, U6.6 (EN)
- new net: R39.1, U6.8 (FB)
- new net: C36.1, C37.1, D3.1 (K), R36.1, U6.2 (VIN)
- new net: D1.2 (A), F1.2
- new net: R38.1, U6.1 (PG)
- new net: R25.1, U4.8 (FB)
- new net: D4.2 (A), JP1.2 (B)
- new net: C24.1, U4.4 (GND)
- new net: C24.2, U4.7 (SS)
- new net: D3.2 (A), F3.2
Other:
- removed sheet Motor1_Power
- removed sheet Motor2_Power1
- removed sheet Sensors_Power
- note added: "Motor 1 Power"
- note added: "Motor 2 Power"
- note added: "Sensor Power"
- moved on the sheet: H1, H2, H3, H4, J4

Commit message: brain fix and almost done with power board layout
Parts:
- renumbered C36 to C1, C39 to C10, C25 to C11, C32 to C12, C40 to C13, C26 to C14, C33 to C15, C41 to C16, C27 to C17, C34 to C18, C42 to C19, C22 to C2, C28 to C20, C35 to C21, C29 to C3, C37 to C4, C23 to C5, C30 to C6, C38 to C7, C24 to C8, C31 to C9, D2 to D1, D3 to D2, D1 to D3, D5 to D4, D6 to D5, D4 to D6, J4 to J1, J6 to J2, J5 to J3, J7 to J4, JP3 to JP1, JP1 to JP3, L3 to L1, L1 to L3, R36 to R1, R25 to R10, R31 to R11, R32 to R12, R40 to R13, R41 to R14, R26 to R15, R27 to R16, R33 to R17, R34 to R18, R28 to R19, R37 to R2, R42 to R20, R35 to R21, R22 to R3, R23 to R4, R29 to R5, R30 to R6, R38 to R7, R39 to R8, R24 to R9, TP4 to TP3, TP3 to TP4, U6 to U1, U4 to U2, U5 to U3
