File: Hardware/power_v1.0/power_v1.0.kicad_pcb (KiCad board)
At the start: 2 copper layers, 0 parts

Commit message: brain fix and almost done with power board layout
Parts:
- added C1: 22uF, Capacitor_SMD:C_0805_2012Metric, F.Cu at (130.2, 110.8)
- added C10: 0.1uF, Capacitor_SMD:C_0603_1608Metric, F.Cu at (141.6, 114.1)
- added C11: 0.1uF, Capacitor_SMD:C_0603_1608Metric, F.Cu at (141.6, 89.2)
- added C12: 0.1uF, Capacitor_SMD:C_0603_1608Metric, F.Cu at (142.0, 65.2)
- added C13: 22uF, Capacitor_SMD:C_0805_2012Metric, F.Cu at (144.9, 114.0)
- added C14: 22uF, Capacitor_SMD:C_0805_2012Metric, F.Cu at (146.0, 87.9)
- added C15: 22uF, Capacitor_SMD:C_0805_2012Metric, F.Cu at (145.7, 64.3)
- added C16: 22uF, Capacitor_SMD:C_0805_2012Metric, F.Cu at (144.9, 118.0)
- added C17: 22uF, Capacitor_SMD:C_0805_2012Metric, F.Cu at (145.9, 92.0)
- added C18: 22uF, Capacitor_SMD:C_0805_2012Metric, F.Cu at (145.7, 68.5)
- added C19: 300pF, Capacitor_SMD:C_0805_2012Metric, F.Cu at (145.0, 110.0)
- added C2: 22uF, Capacitor_SMD:C_0805_2012Metric, F.Cu at (129.6, 84.9)
- added C20: 300pF, Capacitor_SMD:C_0805_2012Metric, F.Cu at (145.9, 83.4)
- added C21: 300pF, Capacitor_SMD:C_0805_2012Metric, F.Cu at (145.7, 60.5)
- added C3: 22uF, Capacitor_SMD:C_0805_2012Metric, F.Cu at (133.5, 62.0)
- added C4: 0.1uF, Capacitor_SMD:C_0603_1608Metric, F.Cu at (133.4, 110.6)
- added C5: 0.1uF, Capacitor_SMD:C_0603_1608Metric, F.Cu at (133.3, 84.7)
- added C6: 0.1uF, Capacitor_SMD:C_0603_1608Metric, F.Cu at (130.3, 61.9)
- added C7: 22nF, Capacitor_SMD:C_0805_2012Metric, F.Cu at (137.0, 115.2)
- added C8: 22nF, Capacitor_SMD:C_0805_2012Metric, F.Cu at (137.6, 89.6)
- added C9: 22nF, Capacitor_SMD:C_0805_2012Metric, F.Cu at (137.6, 65.5)
- added D1: D_Schottky, VS_30BQ015_M3_9AT:VS_30BQ015_M3_9AT, F.Cu at (116.2, 83.9)
- added D2: D_Schottky, VS_30BQ015_M3_9AT:VS_30BQ015_M3_9AT, F.Cu at (116.0, 109.9)
- added D3: D_Schottky, VS_30BQ015_M3_9AT:VS_30BQ015_M3_9AT, F.Cu at (116.8, 60.1)
- added D4: D_Schottky, VS_30BQ015_M3_9AT:VS_30BQ015_M3_9AT, F.Cu at (166.2, 85.2)
- added D5: D_Schottky, VS_30BQ015_M3_9AT:VS_30BQ015_M3_9AT, F.Cu at (165.5, 112.9)
- added D6: D_Schottky, VS_30BQ015_M3_9AT:VS_30BQ015_M3_9AT, F.Cu at (165.8, 62.4)
- added F1: Fuse, 4628:FUSE_4628, F.Cu at (97.2, 60.1)
- added F2: Fuse, 4628:FUSE_4628, F.Cu at (97.4, 84.0)
- added F3: Fuse, 4628:FUSE_4628, F.Cu at (97.2, 109.8)
- added H1: MountingHole, MountingHole:MountingHole_3.2mm_M3, F.Cu at (83.6, 47.6)
- added H2: MountingHole, MountingHole:MountingHole_3.2mm_M3, F.Cu at (176.4, 47.6)
- added H3: MountingHole, MountingHole:MountingHole_3.2mm_M3, F.Cu at (83.6, 140.4)
- added H4: MountingHole, MountingHole:MountingHole_3.2mm_M3, F.Cu at (176.4, 140.4)
- added J1: 12V IN, Connector_Molex:Molex_KK-254_AE-6410-02A_1x02_P2.54mm_Vertical, F.Cu at (86.0, 126.1)
- added J2: Sensor_Power, Connector_Molex:Molex_KK-254_AE-6410-02A_1x02_P2.54mm_Vertical, F.Cu at (176.5, 62.3)
- added J3: Motor1_Power, Connector_Molex:Molex_KK-254_AE-6410-02A_1x02_P2.54mm_Vertical, F.Cu at (176.5, 85.2)
- added J4: Motor2_Power, Connector_Molex:Molex_KK-254_AE-6410-02A_1x02_P2.54mm_Vertical, F.Cu at (176.5, 112.9)
- added JP1: SolderJumper_2_Bridged, Jumper:SolderJumper-2_P1.3mm_Bridged_RoundedPad1.0x1.5mm, F.Cu at (158.2, 112.9)
- added JP2: SolderJumper_2_Bridged, Jumper:SolderJumper-2_P1.3mm_Bridged_RoundedPad1.0x1.5mm, F.Cu at (159.2, 85.2)
- added JP3: SolderJumper_2_Bridged, Jumper:SolderJumper-2_P1.3mm_Bridged_RoundedPad1.0x1.5mm, F.Cu at (158.5, 62.4)
- added L1: 6.8uH, 7447786006:WE-PD_6050R, F.Cu at (137.6, 121.2)
- added L2: 6.8uH, 7447786006:WE-PD_6050R, F.Cu at (137.7, 95.9)
- added L3: 6.8uH, 7447786006:WE-PD_6050R, F.Cu at (138.4, 72.0)
- added R1: 191k, Resistor_SMD:R_1210_3225Metric, F.Cu at (124.7, 111.3)
- added R10: 10k, Resistor_SMD:R_1206_3216Metric, F.Cu at (142.0, 79.8)
- added R11: 10k, Resistor_SMD:R_1206_3216Metric, F.Cu at (137.2, 56.7)
- added R12: 10k, Resistor_SMD:R_1206_3216Metric, F.Cu at (142.5, 56.7)
- added R13: 90.9k, Resistor_SMD:R_1206_3216Metric, F.Cu at (150.0, 111.0)
- added R14: 10k, Resistor_SMD:R_1206_3216Metric, F.Cu at (150.0, 116.7)
- added R15: 90.9k, Resistor_SMD:R_1206_3216Metric, F.Cu at (150.7, 84.8)
- added R16: 10k, Resistor_SMD:R_1206_3216Metric, F.Cu at (150.7, 90.1)
- added R17: 90.9k, Resistor_SMD:R_1206_3216Metric, F.Cu at (150.3, 60.8)
- added R18: 10k, Resistor_SMD:R_1206_3216Metric, F.Cu at (150.3, 65.9)
- added R19: 100k, Resistor_SMD:R_0805_2012Metric, F.Cu at (154.9, 86.2)
- added R2: 49.9k, Resistor_SMD:R_2512_6332Metric, F.Cu at (124.7, 118.7)
- added R20: 100k, Resistor_SMD:R_0805_2012Metric, F.Cu at (153.8, 113.8)
- added R21: 100k, Resistor_SMD:R_0805_2012Metric, F.Cu at (153.8, 63.1)
- added R3: 191k, Resistor_SMD:R_1210_3225Metric, F.Cu at (124.8, 85.4)
- added R4: 49.9k, Resistor_SMD:R_2512_6332Metric, F.Cu at (124.9, 92.5)
- added R5: 191k, Resistor_SMD:R_1210_3225Metric, F.Cu at (125.0, 61.6)
- added R6: 49.9k, Resistor_SMD:R_2512_6332Metric, F.Cu at (125.1, 68.3)
- added R7: 10k, Resistor_SMD:R_1206_3216Metric, F.Cu at (135.0, 106.4)
- added R8: 10k, Resistor_SMD:R_1206_3216Metric, F.Cu at (142.5, 106.3)
- added R9: 10k, Resistor_SMD:R_1206_3216Metric, F.Cu at (135.3, 79.8)
- added TP1: 12V, TestPoint:TestPoint_Keystone_5010-5014_Multipurpose, F.Cu at (93.3, 48.8)
- added TP2: GND, TestPoint:TestPoint_Keystone_5010-5014_Multipurpose, F.Cu at (176.6, 123.0)
- added TP3: Motor1_Power, TestPoint:TestPoint_Keystone_5010-5014_Multipurpose, F.Cu at (158.5, 77.0)
- added TP4: Motor2_Power, TestPoint:TestPoint_Keystone_5010-5014_Multipurpose, F.Cu at (157.5, 104.5)
- added TP5: Sensor_Power, TestPoint:TestPoint_Keystone_5010-5014_Multipurpose, F.Cu at (158.0, 53.0)
- added U1: MP2338GTL-Z, MP2338GTL-Z:SOT583_MP2338_MNP, F.Cu at (138.0, 111.0)
- added U2: MP2338GTL-Z, MP2338GTL-Z:SOT583_MP2338_MNP, F.Cu at (137.4, 84.2)
- added U3: MP2338GTL-Z, MP2338GTL-Z:SOT583_MP2338_MNP, F.Cu at (138.0, 61.3)
Routing:
- net Net-(JP2-A): track 0.00 -> 44.3 mm
- net Net-(JP3-A): track 0.00 -> 43.5 mm
- net Net-(JP1-A): track 0.00 -> 42.6 mm
- net GND: track 0.00 -> 42.5 mm
- net Net-(D2-K): track 0.00 -> 18.3 mm
- net Net-(D3-K): track 0.00 -> 17.7 mm
- net Net-(D1-K): track 0.00 -> 17.2 mm
- net +12V: track 0.00 -> 15.4 mm
- net Net-(U3-BST): track 0.00 -> 14.5 mm
- net Net-(U2-BST): track 0.00 -> 14.5 mm
- net Net-(C20-Pad2): track 0.00 -> 14.4 mm
- net Net-(C19-Pad2): track 0.00 -> 13.8 mm
- net Net-(C21-Pad2): track 0.00 -> 12.8 mm
- net Net-(U1-BST): track 0.00 -> 12.1 mm
- net Net-(U3-EN): track 0.00 -> 8.29 mm, vias 0 -> 2
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- added copper zone on F.Cu, net +12V
- added copper zone on F.Cu, net GND
Other:
- board outline added: 100 x 100 mm
- board text added: "+12V"
- board text added: "+12V IN"
- board text added: "+5V OUT A"
- board text added: "+5V OUT B"
- board text added: "+5V OUT C"
- board text added: "GND"
- board text added: "PAWFEAST: FOOD ON DEMAND Group 30 v1.0"
- board text added: "Sensor 1 Power"
- board text added: "Sensor 2 Power"
- board text added: "Sensor 3 Power"

Commit message: power board done
Parts:
- moved C12 1.53 mm to (140.7, 64.3), turned to -90 degrees
- moved C11 1.18 mm to (141.0, 88.2), turned to -90 degrees
- moved L1 0.88 mm to (137.5, 122.1)
- moved C8 0.83 mm to (137.6, 88.7)
- turned C10 to -90 degrees
Routing:
- net Net-(JP2-A): track 44.3 -> 74.5 mm, vias 0 -> 3
- net Net-(JP1-A): track 42.6 -> 71.0 mm, vias 0 -> 3
- net Net-(JP3-A): track 43.5 -> 69.0 mm, vias 0 -> 4
- net Net-(U3-EN): track 8.29 -> 29.9 mm
- net Net-(U2-EN): track 7.83 -> 25.0 mm
- net Net-(U1-EN): track 7.36 -> 22.5 mm
- net Net-(U1-SW): track 2.19 -> 16.1 mm, vias 1 -> 0
- net Net-(U2-SW): track 1.75 -> 15.2 mm, vias 1 -> 0
- net Net-(U3-SW): track 1.80 -> 14.7 mm, vias 1 -> 0
- net Net-(U2-SS): track 2.90 -> 14.6 mm, vias 1 -> 2
- net Net-(U1-SS): track 2.09 -> 10.6 mm, vias 1 -> 2
- net Net-(U3-SS): track 3.99 -> 12.2 mm, vias 1 -> 2
- net Net-(U1-BST): track 12.1 -> 15.0 mm
- net Net-(U2-BST): track 14.5 -> 16.0 mm
- net Net-(U2-GND): track 4.60 -> 3.70 mm
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- added copper zone on B.Cu, net +12V
- added copper zone on B.Cu, net GND
