File: Hardware/MotorDriver_v1.0/MotorDriver_v1.0.kicad_sch (KiCad schematic)
At the start: 0 parts

Commit message: updated motor driver
Parts:
- added C1, C2, C5: 33uF, Capacitor_SMD:C_0805_2012Metric, symbol device:C_Small
- added C3: 10uF, Capacitor_SMD:C_0805_2012Metric, symbol device:C_Small
- added C4, C7, C8: 0.1uF, Capacitor_SMD:C_0805_2012Metric, symbol device:C_Small
- added C6: 4.7uF, Capacitor_SMD:C_0603_1608Metric, symbol device:C_Small
- added C9: 0.47uF, Capacitor_SMD:C_0805_2012Metric, symbol device:C_Small
- added H1, H2, H3, H4: MountingHole, MountingHole:MountingHole_3.2mm_M3, symbol Mechanical:MountingHole
- added J1, J2, J3, J4: Conn_01x02, Connector_Molex:Molex_KK-254_AE-6410-02A_1x02_P2.54mm_Vertical, symbol Connector_Generic:Conn_01x02
- added J5: Conn_01x04, Connector_Molex:Molex_KK-254_AE-6410-04A_1x04_P2.54mm_Vertical, symbol Connector_Generic:Conn_01x04
- added JP1, JP2, JP3: SolderJumper_2_Bridged, Jumper:SolderJumper-2_P1.3mm_Bridged_RoundedPad1.0x1.5mm, symbol Jumper:SolderJumper_2_Bridged
- added R1, R2: 0.10, Resistor_SMD:R_1206_3216Metric, symbol device:R
- added R3: 10k, Capacitor_SMD:C_0805_2012Metric, symbol device:R
- added R4: 1M, Resistor_SMD:R_0603_1608Metric, symbol device:R
- added RV1: 10k, Capacitor_SMD:C_0805_2012Metric, symbol Device:R_Potentiometer_US
- added U1: DRV8825PWPR, DRV8825:IC_TPS61196PWPRQ1, symbol DRV8825PWPR:DRV8825PWPR
Connections:
- new net: R1.1, U1.9 (ISENB)
- new net: J5.1 (Pin_1), U1.5 (AOUT1)
- new net: J5.2 (Pin_2), U1.7 (AOUT2)
- new net: J5.3 (Pin_3), U1.10 (BOUT1)
- new net: J5.4 (Pin_4), U1.8 (BOUT2)
- new net: C4.2, R4.1, U1.3 (VCP)
- new net: RV1.2, U1.12 (AVREF), U1.13 (BVREF)
- new net: C3.1, U1.1 (CP1)
- new net: C3.2, U1.2 (CP2)
- new net: JP3.1 (A), U1.18 (NFAULT)
- new net: JP3.2 (B), R3.1
- new net: R2.1, U1.6 (ISENA)
- new net: JP2.2 (B), U1.17 (NSLEEP)
- new net: JP1.2 (B), U1.16 (~{NRESET})
- new net +12V: C1.1, C2.1, C4.1, C5.1, C6.1, C7.1, C8.1, J4.1 (Pin_1), R4.2, U1.11 (VMB), U1.4 (VMA)
- new net +3V3: C9.2, J3.1 (Pin_1), RV1.1, U1.15 (V3P3OUT)
- new net +5V: J2.1 (Pin_1), JP1.1 (A), JP2.1 (A), R3.2
- new net DIR: J1.2 (Pin_2), U1.20 (DIR)
- new net GND: C1.2, C2.2, C5.2, C6.2, C7.2, C8.2, C9.1, J2.2 (Pin_2), J3.2 (Pin_2), J4.2 (Pin_2), R1.2, R2.2, RV1.3, U1.14 (GND), U1.28 (GND)
- new net STP: J1.1 (Pin_1), U1.22 (STEP)
- no-connect marks 0 -> 6
Other:
- note added: "Power Connectors"
