File: Hardware/powerLV_v1.0/powerLV_v1.0.kicad_pcb (KiCad board)
At the start: 2 copper layers, 100 x 100 mm, 56 parts, among them J1 Barrel_Jack, J2 12V IN, J3 3v3 Backup, J4 3v3, J5 5V OUT, U1 MP2338GTL-Z, U2 MP2315SGJ-Z, U3 AMS1117-3.3

Commit message: small change to powerLV
Parts:
- moved J1 12.4 mm to (94.3, 106.0), turned to -90 degrees
Routing:
- net +5V: track 25.1 -> 14.4 mm
Changed lines of the file:
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@@
   )
   (footprint "Connector_BarrelJack:BarrelJack_CUI_PJ-102AH_Horizontal" (layer "F.Cu")
-    (at 81.9 107.1 90)
+    (at 94.3 106 -90)
     (descr "Thin-pin DC Barrel Jack, https://cdn-shop.adafruit.com/datasheets/21mmdcjackDatasheet.pdf")
     (tags "Power Jack")
@@
     (fp_line (start 4.5 13.7) (end -4.5 13.7)
       (stroke (width 0.1) (type solid)) (layer "F.Fab"))
-    (pad "1" thru_hole rect (at 0 0 90) (size 2.6 2.6) (drill 1.6) (layers "*.Cu" "*.Mask")
+    (pad "1" thru_hole rect (at 0 0 270) (size 2.6 2.6) (drill 1.6) (layers "*.Cu" "*.Mask")
       (net 20 "+5V") (pintype "passive"))
-    (pad "2" thru_hole circle (at 0 6 90) (size 2.6 2.6) (drill 1.6) (layers "*.Cu" "*.Mask")
+    (pad "2" thru_hole circle (at 0 6 270) (size 2.6 2.6) (drill 1.6) (layers "*.Cu" "*.Mask")
       (net 4 "GND") (pintype "passive"))
-    (pad "3" thru_hole circle (at 4.7 3 90) (size 2.6 2.6) (drill 1.6) (layers "*.Cu" "*.Mask"))
+    (pad "3" thru_hole circle (at 4.7 3 270) (size 2.6 2.6) (drill 1.6) (layers "*.Cu" "*.Mask"))
     (model "${KICAD6_3DMODEL_DIR}/Connector_BarrelJack.3dshapes/BarrelJack_CUI_PJ-102AH_Horizontal.wrl"
       (offset (xyz 0 0 0))
@@
     (effects (font (size 1 1) (thickness 0.15)) (justify left bottom))
   )
-  (gr_text "+5V IN" (at 80.5 99.4) (layer "F.SilkS")
+  (gr_text "+5V IN" (at 80.5 100.2) (layer "F.SilkS")
     (effects (font (size 1.5 1.5) (thickness 0.3) bold) (justify left bottom))
   )
@@
   (segment (start 96.415 88.4) (end 100.89 88.4) (width 0.5) (layer "F.Cu") (net 18))
   (segment (start 106.705 115.6) (end 111.1 115.6) (width 1) (layer "F.Cu") (net 19))
-  (segment (start 84.7 115.6) (end 100.095 115.6) (width 1) (layer "F.Cu") (net 20))
-  (segment (start 81.9 107.1) (end 81.9 112.8) (width 1) (layer "F.Cu") (net 20))
-  (segment (start 81.9 112.8) (end 84.7 115.6) (width 1) (layer "F.Cu") (net 20))
+  (segment (start 97.7 107) (end 97.7 114.8) (width 1) (layer "F.Cu") (net 20))
+  (segment (start 96.7 106) (end 97.7 107) (width 1) (layer "F.Cu") (net 20))
+  (segment (start 94.3 106) (end 96.7 106) (width 1) (layer "F.Cu") (net 20))
+  (segment (start 97.7 114.8) (end 98.4 115.6) (width 1) (layer "F.Cu") (net 20))
+  (segment (start 98.4 115.6) (end 100.095 115.6) (width 1) (layer "F.Cu") (net 20))
   (segment (start 176.38 111.63) (end 170.63 111.63) (width 0.5) (layer "F.Cu") (net 21))
   (segment (start 170.63 111.63) (end 170.5 111.5) (width 0.5) (layer "F.Cu") (net 21))

Commit message: changed LV
Routing:
- net GND: track 2.35 -> 1.13 mm, vias 55 -> 54
Changed lines of the file:
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@@
   (segment (start 89.14 67.33) (end 89.71 67.9) (width 1) (layer "F.Cu") (net 3))
   (segment (start 88.948 76.3) (end 88.948 76.9) (width 1) (layer "F.Cu") (net 3))
-  (segment (start 131.1 91.1) (end 131.1 89.875) (width 0.25) (layer "F.Cu") (net 4))
   (segment (start 136.64745 90.69745) (end 136.65 90.7) (width 0.25) (layer "F.Cu") (net 4))
   (segment (start 136.64745 89.574999) (end 136.64745 90.69745) (width 0.25) (layer "F.Cu") (net 4))
@@
   (via (at 100 95) (size 0.8) (drill 0.4) (layers "F.Cu" "B.Cu") (free) (net 4))
   (via (at 120 125) (size 0.8) (drill 0.4) (layers "F.Cu" "B.Cu") (free) (net 4))
-  (via (at 131.1 91.1) (size 0.8) (drill 0.4) (layers "F.Cu" "B.Cu") (free) (net 4))
   (via (at 155 115) (size 0.8) (drill 0.4) (layers "F.Cu" "B.Cu") (free) (net 4))
   (via (at 175 125) (size 0.8) (drill 0.4) (layers "F.Cu" "B.Cu") (free) (net 4))
