File: Hardware/MotorDriver_v1.5/new_MotorDriver_v1.5_NEW.kicad_sch (KiCad schematic)
At the start: 27 parts, among them J1 Conn_01x02, J2 Conn_01x02, J3 Conn_01x02, J4 Conn_01x02, J5 Conn_01x04, U1 DRV8825PWPR

Commit message: updated motor
yes
Parts:
- removed C1: 33uF, Capacitor_SMD:C_0805_2012Metric, symbol device:C_Small
- removed C6: 4.7uF, Capacitor_SMD:C_0603_1608Metric, symbol device:C_Small
- C2: value 33uF -> 100uF; footprint Capacitor_SMD:C_0805_2012Metric -> Capacitor_SMD:CP_Elec_6.3x5.8
- C5: value 33uF -> 4.7uF
- R3: footprint Capacitor_SMD:C_0805_2012Metric -> Resistor_SMD:R_0805_2012Metric
- RV1: footprint Capacitor_SMD:C_0805_2012Metric -> Potentiometer_THT:Potentiometer_Bourns_PTV09A-1_Single_Vertical
Connections:
- net at J5.1 (Pin_1): now also U1.7 (AOUT2); no longer U1.5 (AOUT1)
- net at J5.2 (Pin_2): now also U1.5 (AOUT1); no longer U1.7 (AOUT2)
Changed lines of the file:
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@@
 	)
 	(junction
-		(at 110.49 137.16)
-		(diameter 0)
-		(color 0 0 0 0)
-	)
-	(junction
 		(at 100.33 142.24)
 		(diameter 0)
@@
 	)
 	(junction
-		(at 110.49 142.24)
-		(diameter 0)
-		(color 0 0 0 0)
-	)
-	(junction
 		(at 102.87 123.19)
 		(diameter 0)
@@
 	(wire
 		(pts
+			(xy 149.86 74.93) (xy 149.86 72.39)
+		)
+		(stroke
+			(width 0)
+			(type default)
+		)
+	)
+	(wire
+		(pts
 			(xy 100.33 142.24) (xy 100.33 146.05)
 		)
@@
 	(wire
 		(pts
-			(xy 53.34 93.98) (xy 53.34 95.25)
+			(xy 148.59 72.39) (xy 148.59 73.66)
 		)
 		(stroke
@@
 	(wire
 		(pts
-			(xy 148.59 82.55) (xy 185.42 82.55)
+			(xy 53.34 93.98) (xy 53.34 95.25)
 		)
 		(stroke
@@
 	(wire
 		(pts
-			(xy 158.75 90.17) (xy 158.75 91.44)
+			(xy 148.59 82.55) (xy 185.42 82.55)
 		)
 		(stroke
@@
 	(wire
 		(pts
-			(xy 110.49 142.24) (xy 121.92 142.24)
+			(xy 158.75 90.17) (xy 158.75 91.44)
 		)
 		(stroke
@@
 	(wire
 		(pts
+			(xy 149.86 72.39) (xy 151.13 72.39)
+		)
+		(stroke
+			(width 0)
+			(type default)
+		)
+	)
+	(wire
+		(pts
 			(xy 102.87 123.19) (xy 102.87 124.46)
 		)
@@
 	(wire
 		(pts
-			(xy 148.59 74.93) (xy 151.13 74.93)
-		)
-		(stroke
-			(width 0)
-			(type default)
-		)
-	)
-	(wire
-		(pts
-			(xy 148.59 72.39) (xy 151.13 72.39)
-		)
-		(stroke
-			(width 0)
-			(type default)
-		)
-	)
-	(wire
-		(pts
 			(xy 106.68 82.55) (xy 113.03 82.55)
 		)
@@
 	(wire
 		(pts
-			(xy 110.49 120.65) (xy 110.49 124.46)
+			(xy 148.59 74.93) (xy 149.86 74.93)
 		)
 		(stroke
@@
 	(wire
 		(pts
-			(xy 148.59 125.73) (xy 152.4 125.73)
+			(xy 110.49 120.65) (xy 110.49 124.46)
 		)
 		(stroke
@@
 	(wire
 		(pts
-			(xy 106.68 97.79) (xy 113.03 97.79)
+			(xy 148.59 125.73) (xy 152.4 125.73)
 		)
 		(stroke
@@
 	(wire
 		(pts
-			(xy 53.34 106.68) (xy 53.34 107.95)
+			(xy 106.68 97.79) (xy 113.03 97.79)
 		)
 		(stroke
@@
 	(wire
 		(pts
-			(xy 113.03 111.76) (xy 97.79 111.76)
+			(xy 53.34 106.68) (xy 53.34 107.95)
 		)
 		(stroke
@@
 	(wire
 		(pts
-			(xy 91.44 142.24) (xy 100.33 142.24)
+			(xy 113.03 111.76) (xy 97.79 111.76)
 		)
 		(stroke
@@
 	(wire
 		(pts
-			(xy 110.49 137.16) (xy 121.92 137.16)
+			(xy 151.13 74.93) (xy 151.13 73.66)
 		)
 		(stroke
@@
 	(wire
 		(pts
-			(xy 91.44 137.16) (xy 100.33 137.16)
+			(xy 41.91 104.14) (xy 55.88 104.14)
 		)
 		(stroke
@@
 	(wire
 		(pts
-			(xy 41.91 104.14) (xy 55.88 104.14)
+			(xy 102.87 123.19) (xy 97.79 123.19)
 		)
 		(stroke
@@
 	(wire
 		(pts
-			(xy 102.87 123.19) (xy 97.79 123.19)
+			(xy 55.88 106.68) (xy 53.34 106.68)
 		)
 		(stroke
@@
 	(wire
 		(pts
-			(xy 55.88 106.68) (xy 53.34 106.68)
+			(xy 100.33 137.16) (xy 110.49 137.16)
 		)
 		(stroke
@@
 	(wire
 		(pts
-			(xy 100.33 137.16) (xy 110.49 137.16)
+			(xy 100.33 95.25) (xy 100.33 91.44)
 		)
 		(stroke
@@
 	(wire
 		(pts
-			(xy 100.33 95.25) (xy 100.33 91.44)
+			(xy 151.13 73.66) (xy 148.59 73.66)
 		)
 		(stroke
@@
 	)
 	(symbol
-		(lib_id "device:C_Small")
-		(at 121.92 139.7 0)
-		(unit 1)
-		(exclude_from_sim no)
-		(in_bom yes)
-		(on_board yes)
-		(dnp no)
-		(fields_autoplaced yes)
-		(property "Reference" "C6"
-			(at 124.46 138.4362 0)
-			(effects
-				(font
-					(size 1.27 1.27)
-				)
-				(justify left)
-			)
-		)
-		(property "Value" "4.7uF"
-			(at 124.46 140.9762 0)
-			(effects
-				(font
-					(size 1.27 1.27)
-				)
-				(justify left)
-			)
-		)
-		(property "Footprint" "Capacitor_SMD:C_0603_1608Metric"
-			(at 121.92 139.7 0)
-			(effects
-				(font
-					(size 1.27 1.27)
-				)
-				(hide yes)
-			)
-		)
-		(property "Datasheet" "~"
-			(at 121.92 139.7 0)
-			(effects
-				(font
-					(size 1.27 1.27)
-				)
-				(hide yes)
-			)
-		)
-		(property "Description" "Unpolarized capacitor, small symbol"
-			(at 121.92 139.7 0)
-			(effects
-				(font
-					(size 1.27 1.27)
-				)
-				(hide yes)
-			)
-		)
-		(pin "2"
-		)
-		(pin "1"
-		)
-		(instances
-			(project ""
-				(path "/1e1b062d-fad0-427c-a622-c5b8a80b5268"
-					(reference "C6")
-					(unit 1)
-				)
-			)
-		)
-	)
-	(symbol
 		(lib_id "power:GND")
 		(at 172.72 72.39 0)
@@
 			)
 		)
-		(property "Footprint" "Capacitor_SMD:C_0805_2012Metric"
+		(property "Footprint" "Potentiometer_THT:Potentiometer_Bourns_PTV09A-1_Single_Vertical"
 			(at 93.98 78.74 0)
 			(effects
@@
 	)
 	(symbol
-		(lib_id "device:C_Small")
-		(at 91.44 139.7 0)
-		(unit 1)
-		(exclude_from_sim no)
-		(in_bom yes)
-		(on_board yes)
-		(dnp no)
-		(property "Reference" "C1"
-			(at 85.852 138.176 0)
-			(effects
-				(font
-					(size 1.27 1.27)
-				)
-				(justify left)
-			)
-		)
-		(property "Value" "33uF"
-			(at 85.344 141.478 0)
-			(effects
-				(font
-					(size 1.27 1.27)
-				)
-				(justify left)
-			)
-		)
-		(property "Footprint" "Capacitor_SMD:C_0805_2012Metric"
-			(at 91.44 139.7 0)
-			(effects
-				(font
-					(size 1.27 1.27)
-				)
-				(hide yes)
-			)
-		)
-		(property "Datasheet" "~"
-			(at 91.44 139.7 0)
-			(effects
-				(font
-					(size 1.27 1.27)
-				)
-				(hide yes)
-			)
-		)
-		(property "Description" "Unpolarized capacitor, small symbol"
-			(at 91.44 139.7 0)
-			(effects
-				(font
-					(size 1.27 1.27)
-				)
-				(hide yes)
-			)
-		)
-		(pin "1"
-		)
-		(pin "2"
-		)
-		(instances
-			(project ""
-				(path "/1e1b062d-fad0-427c-a622-c5b8a80b5268"
-					(reference "C1")
-					(unit 1)
-				)
-			)
-		)
-	)
-	(symbol
 		(lib_id "power:GND")
 		(at 152.4 125.73 0)
@@
 			)
 		)
-		(property "Value" "33uF"
+		(property "Value" "100uF"
 			(at 102.87 140.9762 0)
 			(effects
@@
 			)
 		)
-		(property "Footprint" "Capacitor_SMD:C_0805_2012Metric"
+		(property "Footprint" "Capacitor_SMD:CP_Elec_6.3x5.8"
 			(at 100.33 139.7 0)
 			(effects
@@
 			)
 		)
-		(property "Value" "33uF"
+		(property "Value" "4.7uF"
 			(at 113.03 140.9762 0)
 			(effects
@@
 			)
 		)
-		(property "Footprint" "Capacitor_SMD:C_0805_2012Metric"
+		(property "Footprint" "Resistor_SMD:R_0805_2012Metric"
 			(at 201.93 84.328 90)
 			(effects
