File: Hardware/brain_v2.0/brain_v2.0.kicad_pcb (KiCad board)
At the start: 2 copper layers, 100 x 100 mm, 84 parts, among them J1 Conn_01x02, J10 RFID, J11 Conn_01x05, J12 Conn_01x02, J13 Conn_01x02, J14 Conn_01x02, J15 Conn_01x04, J16 Conn_01x04, J2 Conn_01x02, J3 Conn_01x03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

Commit message: creating PDS board and update other boards
Other:
- board text added: "PAWFEAST: FOOD ON DEMAND Group 30 Brain v2.0"
Changed lines of the file:
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@@
     (effects (font (size 1 1) (thickness 0.15)) (justify left bottom))
+  )
+  (gr_text "PAWFEAST: FOOD ON DEMAND\nGroup 30 \nBrain v2.0" (at 116.3 118) (layer "F.SilkS")
+    (effects (font (size 2 2) (thickness 0.3)) (justify left bottom))
   )
   (gr_text "3v3 Backup" (at 101.8 58.24) (layer "F.SilkS")
