File: Hardware/PDS_v1.0/PDS_v1.0.kicad_pcb (KiCad board)
At the start: 2 copper layers, 28 parts, among them J1 Conn_01x02, J10 Conn_01x02, J11 Conn_01x02, J12 Conn_01x02, J13 Conn_01x04, J14 Conn_01x04, J15 Conn_01x03, J2 Conn_01x02, J3 Conn_01x02, J4 Conn_01x02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

Commit message: PDS done
Parts:
- added H1: MountingHole, MountingHole:MountingHole_3.2mm_M3, F.Cu at (64.2, 41.0)
- added H2: MountingHole, MountingHole:MountingHole_3.2mm_M3, F.Cu at (157.0, 40.8)
- added H3: MountingHole, MountingHole:MountingHole_3.2mm_M3, F.Cu at (157.0, 63.8)
- added H4: MountingHole, MountingHole:MountingHole_3.2mm_M3, F.Cu at (64.0, 63.8)
- added J16: Conn_01x02, Connector_Molex:Molex_KK-254_AE-6410-02A_1x02_P2.54mm_Vertical, F.Cu at (129.0, 63.8)
- C1, C2, C3, R1, R2, R3, R4, R5: moved to B.Cu
- J1, J2: value Conn_01x02 -> Conn_01x04; footprint Connector_Molex:Molex_KK-254_AE-6410-03A_1x03_P2.54mm_Vertical -> Connector_Molex:Molex_KK-254_AE-6410-04A_1x04_P2.54mm_Vertical
- J10, J11, J12, J3, J4, J5, J6, J8, J9: footprint Connector_Molex:Molex_KK-254_AE-6410-03A_1x03_P2.54mm_Vertical -> Connector_Molex:Molex_KK-254_AE-6410-02A_1x02_P2.54mm_Vertical
- J13, J14: value Conn_01x04 -> Conn_01x02; footprint Connector_Molex:Molex_KK-254_AE-6410-04A_1x04_P2.54mm_Vertical -> Connector_Molex:Molex_KK-254_AE-6410-02A_1x02_P2.54mm_Vertical
- J15: value Conn_01x03 -> Conn_01x02; footprint Connector_Molex:Molex_KK-254_AE-6410-03A_1x03_P2.54mm_Vertical -> Connector_Molex:Molex_KK-254_AE-6410-02A_1x02_P2.54mm_Vertical
- J7: value Conn_01x02 -> Conn_01x03
- moved TP1 115.8 mm to (79.0, 40.8)
- moved TP2 104.1 mm to (105.0, 40.7)
- moved TP3 98.5 mm to (129.5, 40.7)
- moved J8 96.4 mm to (64.0, 54.5), turned to -90 degrees
- moved J3 93.1 mm to (73.0, 40.8), turned to 180 degrees
- moved R5 92.0 mm to (148.7, 45.5), turned to 180 degrees
- moved R4 91.2 mm to (141.3, 45.2), turned to -90 degrees
- moved J9 90.7 mm to (70.2, 63.8)
- moved J10 90.2 mm to (78.5, 63.8)
- moved J5 89.8 mm to (124.0, 40.7), turned to 180 degrees
- moved R3 89.1 mm to (139.2, 45.2), turned to -90 degrees
- moved C4 87.8 mm to (136.8, 49.1), turned to 180 degrees
- moved J4 87.1 mm to (99.5, 40.8), turned to 180 degrees
- moved R2 84.3 mm to (145.8, 45.2), turned to -90 degrees
- moved C3 83.7 mm to (140.8, 49.1)
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Connections:
- J1 pad 1: Net-(J1-Pin_1) -> GND
- J1 pad 2: GND -> Net-(J1-Pin_2)
- J1 pad 3: (no net) -> Net-(J1-Pin_3)
- J10 pad 2: Net-(J10-Pin_2) -> +3V3
- J11 pad 2: Net-(J10-Pin_2) -> +5V
- J12 pad 2: Net-(J10-Pin_2) -> +5V
- J13 pad 2: Net-(J13-Pin_2) -> +5V
- J14 pad 2: Net-(J14-Pin_2) -> +12V
- J15 pad 1: /ADC_DRDY -> GND
- J15 pad 2: /ADC_SCL -> +12V
- J2 pad 2: Net-(J1-Pin_1) -> Net-(J2-Pin_2)
- J2 pad 3: (no net) -> Net-(J2-Pin_3)
- J3 pad 1: GND -> +3V3
- J3 pad 2: Net-(J1-Pin_1) -> GND
- J4 pad 1: Net-(J4-Pin_1) -> +5V
- J5 pad 1: GND -> +12V
- J5 pad 2: Net-(J4-Pin_1) -> GND
- J6 pad 1: GND -> Net-(J6-Pin_1)
- J6 pad 2: Net-(J4-Pin_1) -> Net-(J6-Pin_2)
- J7 pad 1: GND -> /ADC_DRDY
- J7 pad 2: Net-(J4-Pin_1) -> /ADC_SCL
- J7 pad 3: (no net) -> /ADC_SDA
- J8 pad 2: Net-(J1-Pin_1) -> +3V3
- J9 pad 1: Net-(J10-Pin_2) -> GND
- J9 pad 2: GND -> +3V3
- R1 pad 1: Net-(J13-Pin_3) -> Net-(J1-Pin_3)
- R2 pad 1: Net-(J13-Pin_2) -> Net-(J1-Pin_2)
- R3 pad 1: Net-(J14-Pin_3) -> Net-(J2-Pin_3)
- R4 pad 1: Net-(J14-Pin_2) -> Net-(J2-Pin_2)
- TP1 pad 1: Net-(J1-Pin_1) -> +3V3
- TP2 pad 1: Net-(J4-Pin_1) -> +5V
- TP3 pad 1: Net-(J10-Pin_2) -> +12V
- U1 pad 10: unconnected-(U1-XIN-Pad10) -> Net-(J6-Pin_1)
- U1 pad 11: unconnected-(U1-XOUT-Pad11) -> Net-(J6-Pin_2)
Routing:
- net +5V: track 0.00 -> 137.1 mm, vias 0 -> 34
- net +3V3: track 0.00 -> 67.5 mm, vias 0 -> 18
- net +12V: track 0.00 -> 50.4 mm, vias 0 -> 26
- net Net-(J2-Pin_2): track 0.00 -> 32.8 mm, vias 0 -> 1
- net Net-(J2-Pin_3): track 0.00 -> 24.5 mm, vias 0 -> 1
- net /ADC_SDA: track 0.00 -> 9.81 mm
- net /ADC_SCL: track 0.00 -> 9.18 mm
- net /ADC_DRDY: track 0.00 -> 8.81 mm
- net Net-(U1-VIN2P): track 0.00 -> 7.71 mm, vias 0 -> 1
- net Net-(J6-Pin_1): track 0.00 -> 7.36 mm
- net Net-(U1-VIN2N): track 0.00 -> 7.12 mm, vias 0 -> 1
- net Net-(J6-Pin_2): track 0.00 -> 7.09 mm
- net Net-(U1-REFP): track 0.00 -> 6.54 mm, vias 0 -> 1
- net Net-(U1-VIN1P): track 0.00 -> 6.42 mm, vias 0 -> 1
- net Net-(U1-VIN1N): track 0.00 -> 6.09 mm, vias 0 -> 1
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- added copper zone on B.Cu, net +12V
- added copper zone on F.Cu, net +12V
- added copper zone on B.Cu, net +3V3
- added copper zone on F.Cu, net +3V3
- added copper zone on B.Cu, net +5V
- added copper zone on F.Cu, net +5V
- added copper zone on B.Cu, net GND
- added copper zone on F.Cu, net GND
Other:
- board outline added: 100 x 30 mm
- board text added: "PAWFEAST: FOOD ON DEMAND Group 30 | PDS v1.0"

Commit message: fixed silkscreens + readability on PDS
Parts:
- added C5: 470uF, Capacitor_THT:C_Radial_D10.0mm_H12.5mm_P5.00mm, B.Cu at (109.7, 48.4)
- added TP4: TestPoint, TestPoint:TestPoint_Keystone_5010-5014_Multipurpose, F.Cu at (121.2, 51.5)
- added TP5: TestPoint, TestPoint:TestPoint_Keystone_5010-5014_Multipurpose, F.Cu at (126.8, 51.5)
- added TP6: TestPoint, TestPoint:TestPoint_Keystone_5010-5014_Multipurpose, F.Cu at (131.9, 50.6)
Routing:
- net Net-(U1-VIN2P): track 7.71 -> 38.8 mm
- net Net-(U1-VIN2N): track 7.12 -> 38.1 mm
- net /ADC_DRDY: track 8.81 -> 34.2 mm, vias 0 -> 1
- net /ADC_SCL: track 9.18 -> 29.4 mm, vias 0 -> 1
- net /ADC_SDA: track 9.81 -> 27.1 mm, vias 0 -> 1
Other:
- board text added: "+"
- board text added: "+12V"
- board text added: "+12V IN"
- board text added: "+5V"
- board text added: "+5V IN"
- board text added: "-"
- board text added: "1+"
- board text added: "1-"
- board text added: "2+"
- board text added: "2-"
- board text added: "3v3"
- board text added: "3v3 IN"
- board text added: "DRDY"
- board text added: "GND"
- board text added: "SCL"
- board text added: "SDA"
- board text added: "Xin"
- board text added: "Xout"
